File: KiCAD_Project/WxBackpack.kicad_pcb (KiCad board)
At the start: 2 copper layers, 20.4 x 45.1 mm, 56 parts, among them P1 CONN_1, P2 CONN_1, P3 CONN_1, P4 CONN_1, P5 CONN_1, P6 CONN_1, P7 CONN_1, U1 HTU21D, U2 BMP180

Commit message: Finish layout and finalize rev.A boards
Parts:
- added G***: LOGO, LOGO, B.Cu at (217.4, 115.1)
- moved C1 8.54 mm to (217.4, 110.2), turned to 180 degrees
- moved R2 7.08 mm to (217.4, 115.7)
- moved C2 6.75 mm to (217.4, 107.7), turned to 180 degrees
- moved C3 5.08 mm to (217.4, 92.4), turned to 0 degrees
- moved U1 5.08 mm to (217.4, 96.4)
- moved U2 4.31 mm to (223.0, 109.2), turned to 270 degrees
- moved R1 2.94 mm to (217.4, 113.3)
- moved C4 2.94 mm to (223.0, 105.2), turned to 180 degrees
Connections:
- U1 pad 1: (no net) -> SDA
- U1 pad 2: +3.3V -> GND
- U1 pad 3: SCL -> (no net)
- U1 pad 5: GND -> +3.3V
- U1 pad 6: SDA -> SCL
Routing:
- net SDA: track 8.82 -> 54.3 mm, vias 0 -> 2
- net SCL: track 6.57 -> 45.2 mm, vias 0 -> 2
- net GND: track 0.00 -> 38.6 mm, vias 0 -> 5
- net +3.3V: track 51.3 -> 47.3 mm
- net +BATT: track 0.00 -> 2.54 mm
- added copper zone on B.Cu, net GND
- added copper zone on F.Cu, net GND
Other:
- outline, holes or cut-outs redrawn
- board text added: "0"
- board text added: "0.1" Slot"
- board text added: "1"
- board text added: "2"
- board text added: "3"
- board text added: "4"
- board text added: "5"
- board text added: "A0"
- board text added: "A1"
- board text added: "BAT"
- board text added: "GND"
- board text added: "RST"
- board text added: "Rev. A - 2015"
- board text added: "VCC"
